File: hardware/ummon.kicad_sch (KiCad schematic)
At the start: 86 parts, among them J1 Conn_01x08_Pin, J2 Conn_01x05_Pin, J3 Conn_01x04_Pin, J4 Conn_01x04_Pin, J5 Conn_01x04_Pin, P1 Display, Q1 BSS138LT1G, SW1 Reboot, SW2 Flash, SW3 Test Button, SW4 MINI MSK12CO2, U1 ESP32-C6-WROOM-1-N8, U2 SCD41, U3 SGP41, U4 SHT41, U5 AMS1117-3.3

Commit message: :sparkles: E-Paper driver board is now reflecting revision 2.3 including the pwr control
Parts:
- removed J1: Conn_01x08_Pin, Connector_PinHeader_2.54mm:PinHeader_1x08_P2.54mm_Vertical, symbol Connector:Conn_01x08_Pin
- removed L1: 68μH, parts:IND-SMD_L4.0-W4.0_FNR40XXS, symbol parts:FNR4030S680MT
- added C19, C21: 100nF, Capacitor_SMD:C_0805_2012Metric, symbol Device:C_Small
- added C20: 10µF, Capacitor_SMD:C_0805_2012Metric, symbol Device:C_Small
- added J6: Conn_01x09_Pin, Connector_PinHeader_2.54mm:PinHeader_1x09_P2.54mm_Vertical, symbol Connector:Conn_01x09_Pin
- added Q2: AO3401A, parts:SOT-23_L2.9-W1.3-P1.90-LS2.4-BR, symbol parts:AO3401A
- added R17: 100kΩ, Resistor_SMD:R_0805_2012Metric, symbol Device:R_Small
- added R18: 4.7kΩ, Resistor_SMD:R_0805_2012Metric, symbol Device:R_Small
- added U6: 10μH, parts:IND-SMD_L4.5-W4.0, symbol parts:CY43-10UH
- C28: value 1μF/20V -> 1μF/25V
- TP4: value PVGH -> PCP
- TP5: value PVGL -> PSW
Connections:
- net +3.3V: now also C19.1, J6.1 (Pin_1), Q2.2 (S), R17.1; no longer C18.2, C22.2, C27.2, P1.10, P1.9
- net EPD_BUSY: now also J6.8 (Pin_8)
- net EPD_CS: now also J6.5 (Pin_5)
- net EPD_DC: now also J6.6 (Pin_6)
- net EPD_DIN: now also J6.3 (Pin_3)
- net EPD_RST: now also J6.7 (Pin_7)
- net EPD_SCK: now also J6.4 (Pin_4)
- net EPD_VGH: now also C32.2, D2.1 (K), P1.4; no longer C26.2, D2.2 (A), Q1.3 (D)
- net EPD_VGL: now also C36.2, D4.2 (A), P1.2; no longer C26.1, D3.2 (A), D4.1 (K)
- net GND: now also P1.25, P1.26, C20.2, C21.2, J6.2 (Pin_2)
- net EPD_PWR: now reaches U1.23 (IO15)
- net EPD_PWR: now also J6.9 (Pin_9), R18.2
- removed net EPD_PREVGH: C32.2, D2.1 (K), P1.4, TP4.1
- removed net EPD_PREVGL: C36.2, D4.2 (A), P1.2, TP5.1
- new net: C19.2, Q2.1 (G), R17.2, R18.1
- new net EPD_3V3: C18.2, C20.1, C21.1, C22.2, C27.2, P1.10, P1.9, Q2.3 (D), U6.1
- new net EPD_CP: C26.1, D3.2 (A), D4.1 (K), TP4.1
- new net EPD_SW: C26.2, D2.2 (A), Q1.3 (D), TP5.1, U6.2
- no-connect marks 27 -> 24

Commit message: :sparkles: Power LED can now be turned off via firmware
Parts:
- added Q3: AO3401A, parts:SOT-23_L2.9-W1.3-P1.90-LS2.4-BR, symbol parts:AO3401A
- added R19: 100kΩ, Resistor_SMD:R_0805_2012Metric, symbol Device:R_Small
Connections:
- net +3.3V: now also Q3.2 (S); no longer R14.1
- net GND: now also R19.2
- net GPIO5: now reaches U1.5 (IO5)
- net GPIO5: now also Q3.1 (G), R19.1
- new net: Q3.3 (D), R14.1
- no-connect marks 24 -> 23
Other:
- moved on the sheet: C14, C15, C16, C17, U5

Commit message: wip
Parts:
- removed C20: 10µF, Capacitor_SMD:C_0805_2012Metric, symbol Device:C_Small
Connections:
- net EPD_VSL: now reaches C34.2, P1.3
- net EPD_VDD: now reaches C28.2, P1.7
- net EPD_VCOM: now reaches C38.2, P1.1
- net EPD_VSH2: now reaches C24.2, P1.20
- net EPD_VSH: now reaches C30.2, P1.5

Commit message: :sparkles: Completes routing for epd rev 2.3
Parts:
- added TP11: EPD_3V3, TestPoint:TestPoint_Pad_D1.0mm, symbol Connector:TestPoint
Connections:
- net EPD_3V3: now also TP11.1
- net EPD_RESE_0.47O: now reaches R11.2, R13.2, SW4.3
- net EPD_RESE_3O: now reaches R10.2, SW4.1
Other:
- moved on the sheet: R10, R16
Changed lines of the file:
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@@
 	(wire
 		(pts
-			(xy 264.16 25.4) (xy 266.7 25.4)
+			(xy 275.59 25.4) (xy 278.13 25.4)
 		)
 		(stroke
@@
 	(wire
 		(pts
-			(xy 243.84 25.4) (xy 251.46 25.4)
+			(xy 243.84 25.4) (xy 262.89 25.4)
 		)
 		(stroke
@@
 	(wire
 		(pts
-			(xy 256.54 25.4) (xy 259.08 25.4)
+			(xy 267.97 25.4) (xy 270.51 25.4)
 		)
 		(stroke
@@
 		)
 	)
+	(label "EPD_RESE_0.47O"
+		(at 243.84 35.56 0)
+		(effects
+			(font
+				(size 1.27 1.27)
+			)
+			(justify left bottom)
+		)
+	)
 	(label "H_PRESENCE"
 		(at 133.35 158.75 180)
@@
 		)
 	)
-	(label "Reference had a single 3Ω R"
-		(at 250.19 19.05 0)
-		(effects
-			(font
-				(size 0.8382 0.8382)
-				(color 255 0 0 1)
-			)
-			(justify left bottom)
-		)
-	)
 	(label "EPD_VSL"
 		(at 360.68 86.36 0)
@@
 		)
 	)
+	(label "EPD_RESE_3O"
+		(at 245.11 25.4 0)
+		(effects
+			(font
+				(size 1.27 1.27)
+			)
+			(justify left bottom)
+		)
+	)
 	(label "CO2 Sensor"
 		(at 40.64 207.01 0)
@@
 		)
 	)
-	(label "Reference had a single 0.47Ω R"
-		(at 238.76 49.53 0)
-		(effects
-			(font
-				(size 0.8382 0.8382)
-				(color 255 0 0 1)
-			)
-			(justify left bottom)
-		)
-	)
 	(symbol
 		(lib_id "power:+3.3V")
@@
 	)
 	(symbol
+		(lib_id "power:+3.3V")
+		(at 358.14 218.44 180)
+		(unit 1)
+		(body_style 1)
+		(exclude_from_sim no)
+		(in_bom yes)
+		(on_board yes)
+		(in_pos_files yes)
+		(dnp no)
+		(fields_autoplaced yes)
+		(property "Reference" "#PWR064"
+			(at 358.14 214.63 0)
+			(hide yes)
+			(show_name no)
+			(do_not_autoplace no)
+			(effects
+				(font
+					(size 1.27 1.27)
+				)
+			)
+		)
+		(property "Value" "EPD_3V3"
+			(at 358.14 223.52 0)
+			(show_name no)
+			(do_not_autoplace no)
+			(effects
+				(font
+					(size 1.27 1.27)
+				)
+			)
+		)
+		(property "Footprint" ""
+			(at 358.14 218.44 0)
+			(hide yes)
+			(show_name no)
+			(do_not_autoplace no)
+			(effects
+				(font
+					(size 1.27 1.27)
+				)
+			)
+		)
+		(property "Datasheet" ""
+			(at 358.14 218.44 0)
+			(hide yes)
+			(show_name no)
+			(do_not_autoplace no)
+			(effects
+				(font
+					(size 1.27 1.27)
+				)
+			)
+		)
+		(property "Description" "Power symbol creates a global label with name \"+3.3V\""
+			(at 358.14 218.44 0)
+			(hide yes)
+			(show_name no)
+			(do_not_autoplace no)
+			(effects
+				(font
+					(size 1.27 1.27)
+				)
+			)
+		)
+		(pin "1"
+		)
+		(instances
+			(project "ummon"
+				(path "/535d19c6-6731-456b-b7fb-ac6bb0b86499"
+					(reference "#PWR064")
+					(unit 1)
+				)
+			)
+		)
+	)
+	(symbol
 		(lib_id "Device:C_Small")
 		(at 30.48 222.25 0)
@@
 	(symbol
 		(lib_id "Device:R_Small")
-		(at 254 25.4 270)
+		(at 265.43 25.4 270)
 		(unit 1)
 		(body_style 1)
@@
 		(fields_autoplaced yes)
 		(property "Reference" "R10"
-			(at 254 20.32 90)
+			(at 265.43 20.32 90)
 			(show_name no)
 			(do_not_autoplace no)
@@
 		)
 		(property "Value" "2.2Ω"
-			(at 254 22.86 90)
+			(at 265.43 22.86 90)
 			(show_name no)
 			(do_not_autoplace no)
@@
 		)
 		(property "Footprint" "Resistor_SMD:R_0805_2012Metric"
-			(at 254 25.4 0)
+			(at 265.43 25.4 0)
 			(hide yes)
 			(show_name no)
@@
 		)
 		(property "Datasheet" ""
-			(at 254 25.4 0)
+			(at 265.43 25.4 0)
 			(hide yes)
 			(show_name no)
@@
 		)
 		(property "Description" "Resistor, small symbol"
-			(at 254 25.4 0)
+			(at 265.43 25.4 0)
 			(hide yes)
 			(show_name no)
@@
 		)
 		(property "LCSC Part" "C17521"
-			(at 254 25.4 90)
+			(at 265.43 25.4 90)
 			(hide yes)
 			(show_name no)
@@
 	)
 	(symbol
+		(lib_id "Connector:TestPoint")
+		(at 358.14 218.44 0)
+		(unit 1)
+		(body_style 1)
+		(exclude_from_sim no)
+		(in_bom yes)
+		(on_board yes)
+		(in_pos_files yes)
+		(dnp no)
+		(fields_autoplaced yes)
+		(property "Reference" "TP11"
+			(at 360.68 213.8679 0)
+			(show_name no)
+			(do_not_autoplace no)
+			(effects
+				(font
+					(size 1.27 1.27)
+				)
+				(justify left)
+			)
+		)
+		(property "Value" "EPD_3V3"
+			(at 360.68 216.4079 0)
+			(show_name no)
+			(do_not_autoplace no)
+			(effects
+				(font
+					(size 1.27 1.27)
+				)
+				(justify left)
+			)
+		)
+		(property "Footprint" "TestPoint:TestPoint_Pad_D1.0mm"
+			(at 363.22 218.44 0)
+			(hide yes)
+			(show_name no)
+			(do_not_autoplace no)
+			(effects
+				(font
+					(size 1.27 1.27)
+				)
+			)
+		)
+		(property "Datasheet" ""
+			(at 363.22 218.44 0)
+			(hide yes)
+			(show_name no)
+			(do_not_autoplace no)
+			(effects
+				(font
+					(size 1.27 1.27)
+				)
+			)
+		)
+		(property "Description" "test point"
+			(at 358.14 218.44 0)
+			(hide yes)
+			(show_name no)
+			(do_not_autoplace no)
+			(effects
+				(font
+					(size 1.27 1.27)
+				)
+			)
+		)
+		(pin "1"
+		)
+		(instances
+			(project "ummon"
+				(path "/535d19c6-6731-456b-b7fb-ac6bb0b86499"
+					(reference "TP11")
+					(unit 1)
+				)
+			)
+		)
+	)
+	(symbol
 		(lib_id "power:+3.3V")
 		(at 313.69 58.42 0)
@@
 	(symbol
 		(lib_id "Device:R_Small")
-		(at 261.62 25.4 270)
+		(at 273.05 25.4 270)
 		(unit 1)
 		(body_style 1)
@@
 		(fields_autoplaced yes)
 		(property "Reference" "R16"
-			(at 261.62 20.32 90)
+			(at 273.05 20.32 90)
 			(show_name no)
 			(do_not_autoplace no)
@@
 		)
 		(property "Value" "1Ω"
-			(at 261.62 22.86 90)
+			(at 273.05 22.86 90)
 			(show_name no)
 			(do_not_autoplace no)
@@
 		)
 		(property "Footprint" "Resistor_SMD:R_0805_2012Metric"
-			(at 261.62 25.4 0)
+			(at 273.05 25.4 0)
 			(hide yes)
 			(show_name no)
@@
 		)
 		(property "Datasheet" ""
-			(at 261.62 25.4 0)
+			(at 273.05 25.4 0)
 			(hide yes)
 			(show_name no)
@@
 		)
 		(property "Description" "Resistor, small symbol"
-			(at 261.62 25.4 0)
+			(at 273.05 25.4 0)
 			(hide yes)
 			(show_name no)
@@
 		)
 		(property "LCSC Part" "C25271"
-			(at 261.62 25.4 90)
+			(at 273.05 25.4 90)
 			(hide yes)
 			(show_name no)
@@
 	(symbol
 		(lib_id "power:GND")
-		(at 266.7 25.4 0)
+		(at 278.13 25.4 0)
 		(unit 1)
 		(body_style 1)
@@
 		(fields_autoplaced yes)
 		(property "Reference" "#PWR042"
-			(at 266.7 31.75 0)
+			(at 278.13 31.75 0)
 			(hide yes)
 			(show_name no)
@@
 		)
 		(property "Value" "GND"
-			(at 266.7 30.48 0)
+			(at 278.13 30.48 0)
 			(show_name no)
 			(do_not_autoplace no)
@@
 		)
 		(property "Footprint" ""
-			(at 266.7 25.4 0)
+			(at 278.13 25.4 0)
 			(hide yes)
 			(show_name no)
@@
 		)
 		(property "Datasheet" ""
-			(at 266.7 25.4 0)
+			(at 278.13 25.4 0)
 			(hide yes)
 			(show_name no)
@@
 		)
 		(property "Description" "Power symbol creates a global label with name \"GND\" , ground"
-			(at 266.7 25.4 0)
+			(at 278.13 25.4 0)
 			(hide yes)
 			(show_name no)
